File: kicad/Super7Controller/Super7Controller.kicad_pcb (KiCad board)
At the start: 2 copper layers, 49.5 x 25.4 mm, 20 parts, among them P3 CONN_01X13, P4 CONN_01X09, U1 ULN2003A, U2 HiLetgo_ESP-WROOM-32_Developm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

Commit message: correct errors in netlist
Connections:
- U2 pad 10: DCD_2 -> DCD_1
- U2 pad 11: DCD_1 -> DCD_2
- U2 pad 15: DCD_4 -> DCD_3
- U2 pad 9: DCD_3 -> DCD_4
Routing:
- net DCD_4: track 22.1 -> 27.4 mm
- net DCD_3: track 20.0 -> 14.7 mm
- net DCD_1: track 28.8 -> 24.5 mm
- net DCD_2: track 17.4 -> 21.7 mm
Changed lines of the file:
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@@
   (general
     (links 45)
-    (no_connects 4)
+    (no_connects 0)
     (area 69.139999 53.264999 118.820001 78.815001)
     (thickness 1.6)
@@
       (net 27 "Net-(R1-Pad1)"))
     (pad 9 thru_hole oval (at -2.54 11.425) (size 1.2 2) (drill 0.8) (layers *.Cu *.Mask)
-      (net 61 DCD_3))
+      (net 58 DCD_4))
     (pad 29 thru_hole oval (at 0 -11.425) (size 1.2 2) (drill 0.8) (layers *.Cu *.Mask)
       (net 36 "Net-(R10-Pad1)"))
     (pad 10 thru_hole oval (at 0 11.425) (size 1.2 2) (drill 0.8) (layers *.Cu *.Mask)
-      (net 60 DCD_2))
+      (net 59 DCD_1))
     (pad 28 thru_hole oval (at 2.54 -11.425) (size 1.2 2) (drill 0.8) (layers *.Cu *.Mask)
       (net 37 "Net-(R11-Pad1)"))
     (pad 11 thru_hole oval (at 2.54 11.425) (size 1.2 2) (drill 0.8) (layers *.Cu *.Mask)
-      (net 59 DCD_1))
+      (net 60 DCD_2))
     (pad 27 thru_hole oval (at 5.08 -11.425) (size 1.2 2) (drill 0.8) (layers *.Cu *.Mask)
       (net 39 "Net-(R13-Pad1)"))
@@
       (net 57 DCD_5))
     (pad 15 thru_hole oval (at 12.7 11.425) (size 1.2 2) (drill 0.8) (layers *.Cu *.Mask)
-      (net 58 DCD_4))
+      (net 61 DCD_3))
     (pad 23 thru_hole oval (at 15.24 -11.425) (size 1.2 2) (drill 0.8) (layers *.Cu *.Mask)
       (net 56 DCD_6))
@@
   (segment (start 114.0262 63.0222) (end 114.0262 62.946) (width 0.1524) (layer B.Cu) (net 57))
   (segment (start 114.7 63.246) (end 114.0262 63.0222) (width 0.1524) (layer B.Cu) (net 57))
-  (segment (start 106.7 77.025) (end 106.7 77.425) (width 0.1524) (layer B.Cu) (net 58))
-  (segment (start 115.5763 71.4709) (end 106.7 77.025) (width 0.1524) (layer B.Cu) (net 58))
-  (segment (start 115.7549 71.2923) (end 115.5763 71.4709) (width 0.1524) (layer B.Cu) (net 58))
-  (segment (start 115.7549 71.0397) (end 115.7549 71.2923) (width 0.1524) (layer B.Cu) (net 58))
-  (segment (start 115.7549 69.1697) (end 115.7549 71.0397) (width 0.1524) (layer B.Cu) (net 58))
-  (segment (start 115.3738 68.6576) (end 115.7549 69.1697) (width 0.1524) (layer B.Cu) (net 58))
   (segment (start 114.0262 64.816) (end 114.0262 64.8476) (width 0.1524) (layer B.Cu) (net 58))
   (segment (start 114.0262 64.7398) (end 114.0262 64.816) (width 0.1524) (layer B.Cu) (net 58))
@@
   (segment (start 110.3549 68.7523) (end 110.1763 68.9309) (width 0.1524) (layer B.Cu) (net 58))
   (segment (start 110.1763 68.9309) (end 108.4237 68.9911) (width 0.1524) (layer B.Cu) (net 58))
+  (segment (start 91.46 77.025) (end 91.46 77.425) (width 0.1524) (layer B.Cu) (net 58))
+  (segment (start 108.4237 68.9911) (end 91.46 77.025) (width 0.1524) (layer B.Cu) (net 58))
   (segment (start 114.0262 66.086) (end 114.0262 66.1176) (width 0.1524) (layer B.Cu) (net 59))
   (segment (start 114.0262 66.0098) (end 114.0262 66.086) (width 0.1524) (layer B.Cu) (net 59))
   (segment (start 114.7 65.786) (end 114.0262 66.0098) (width 0.1524) (layer B.Cu) (net 59))
   (segment (start 114.0262 66.1176) (end 110.3549 70.0223) (width 0.1524) (layer B.Cu) (net 59))
-  (segment (start 96.54 77.025) (end 96.54 77.425) (width 0.1524) (layer B.Cu) (net 59))
-  (segment (start 98.7052 76.1201) (end 96.54 77.025) (width 0.1524) (layer B.Cu) (net 59))
-  (segment (start 110.1763 71.4709) (end 98.7052 76.1201) (width 0.1524) (layer B.Cu) (net 59))
-  (segment (start 110.3549 71.2923) (end 110.1763 71.4709) (width 0.1524) (layer B.Cu) (net 59))
-  (segment (start 113.2038 67.7169) (end 110.3549 71.2923) (width 0.1524) (layer B.Cu) (net 59))
-  (segment (start 113.6409 67.2798) (end 113.2038 67.7169) (width 0.1524) (layer B.Cu) (net 59))
   (segment (start 110.3549 70.0223) (end 110.1763 70.2009) (width 0.1524) (layer B.Cu) (net 59))
   (segment (start 110.1763 70.2009) (end 108.4237 70.2611) (width 0.1524) (layer B.Cu) (net 59))
-  (segment (start 94 77.025) (end 94 77.425) (width 0.1524) (layer B.Cu) (net 60))
-  (segment (start 108.4237 70.2611) (end 94 77.025) (width 0.1524) (layer B.Cu) (net 60))
+  (segment (start 94 77.025) (end 94 77.425) (width 0.1524) (layer B.Cu) (net 59))
+  (segment (start 108.4237 70.2611) (end 94 77.025) (width 0.1524) (layer B.Cu) (net 59))
+  (segment (start 96.54 77.025) (end 96.54 77.425) (width 0.1524) (layer B.Cu) (net 60))
+  (segment (start 98.7052 76.1201) (end 96.54 77.025) (width 0.1524) (layer B.Cu) (net 60))
+  (segment (start 110.1763 71.4709) (end 98.7052 76.1201) (width 0.1524) (layer B.Cu) (net 60))
+  (segment (start 110.3549 71.2923) (end 110.1763 71.4709) (width 0.1524) (layer B.Cu) (net 60))
+  (segment (start 113.2038 67.7169) (end 110.3549 71.2923) (width 0.1524) (layer B.Cu) (net 60))
+  (segment (start 113.6409 67.2798) (end 113.2038 67.7169) (width 0.1524) (layer B.Cu) (net 60))
   (segment (start 113.95 67.2798) (end 113.6409 67.2798) (width 0.1524) (layer B.Cu) (net 60))
   (segment (start 114.0262 67.2798) (end 113.95 67.2798) (width 0.1524) (layer B.Cu) (net 60))
   (segment (start 114.7 67.056) (end 114.0262 67.2798) (width 0.1524) (layer B.Cu) (net 60))
-  (segment (start 91.46 77.025) (end 91.46 77.425) (width 0.1524) (layer B.Cu) (net 61))
-  (segment (start 108.4237 68.9911) (end 91.46 77.025) (width 0.1524) (layer B.Cu) (net 61))
+  (segment (start 106.7 77.025) (end 106.7 77.425) (width 0.1524) (layer B.Cu) (net 61))
+  (segment (start 115.5763 71.4709) (end 106.7 77.025) (width 0.1524) (layer B.Cu) (net 61))
+  (segment (start 115.7549 71.2923) (end 115.5763 71.4709) (width 0.1524) (layer B.Cu) (net 61))
+  (segment (start 115.7549 71.0397) (end 115.7549 71.2923) (width 0.1524) (layer B.Cu) (net 61))
+  (segment (start 115.7549 69.1697) (end 115.7549 71.0397) (width 0.1524) (layer B.Cu) (net 61))
+  (segment (start 115.3738 68.6576) (end 115.7549 69.1697) (width 0.1524) (layer B.Cu) (net 61))
   (segment (start 115.3738 68.626) (end 115.3738 68.6576) (width 0.1524) (layer B.Cu) (net 61))
   (segment (start 115.3738 68.5498) (end 115.3738 68.626) (width 0.1524) (layer B.Cu) (net 61))
