File: kicad/Super7Controller/Super7Controller.sch (KiCad schematic (older format))
At the start: 20 parts, among them P3 Conn_01x13, P4 Conn_01x09, U1 ULN2003A, U2 HiLetgo_ESP-WROOM-32_Developm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

Commit message: Apply bodge wire fix to controller PCB
Decimal points are no longer connected
Parts:
- removed R4, R9: 120, Resistors_SMD:R_0805_HandSoldering, symbol R
Connections:
- no-connect marks 17 -> 21
Other:
- note added: "Ran out of GPIO outputs to control these pins"
- moved on the sheet: R8
Changed lines of the file:
@@
 Text GLabel 8750 2550 2    50   Input ~ 0
 H_G1
-Text GLabel 5700 2550 0    50   Input ~ 0
+Text GLabel 9500 4050 0    50   Input ~ 0
 H_DP1
 $Comp
@@
 	0    -1   -1   0
 $EndComp
-$Comp
-L R R4
-U 1 1 585D9A03
-P 5850 2550
-F 0 "R4" V 5930 2550 50  0000 C CNN
-F 1 "120" V 5850 2550 50  0000 C CNN
-F 2 "Resistors_SMD:R_0805_HandSoldering" V 5780 2550 50  0001 C CNN
-F 3 "" H 5850 2550 50  0000 C CNN
-	1    5850 2550
-	0    1    -1   0
-$EndComp
 Text GLabel 8750 1850 2    50   Input ~ 0
 H_A2
 Text GLabel 8250 1750 2    50   Input ~ 0
 H_B2
-Text GLabel 5700 2150 0    50   Input ~ 0
+Text GLabel 5700 2550 0    50   Input ~ 0
 H_C2
 Text GLabel 5700 2350 0    50   Input ~ 0
@@
 Text GLabel 6250 2250 0    50   Input ~ 0
 H_G2
-Text GLabel 6250 2050 0    50   Input ~ 0
+Text GLabel 9500 4200 0    50   Input ~ 0
 H_DP2
 $Comp
@@
 L R R8
 U 1 1 585DBA07
-P 5850 2150
-F 0 "R8" V 5930 2150 50  0000 C CNN
-F 1 "120" V 5850 2150 50  0000 C CNN
-F 2 "Resistors_SMD:R_0805_HandSoldering" V 5780 2150 50  0001 C CNN
-F 3 "" H 5850 2150 50  0000 C CNN
-	1    5850 2150
+P 5850 2550
+F 0 "R8" V 5930 2550 50  0000 C CNN
+F 1 "120" V 5850 2550 50  0000 C CNN
+F 2 "Resistors_SMD:R_0805_HandSoldering" V 5780 2550 50  0001 C CNN
+F 3 "" H 5850 2550 50  0000 C CNN
+	1    5850 2550
 	0    1    -1   0
 $EndComp
@@
 F 3 "" H 6400 2250 50  0000 C CNN
 	1    6400 2250
-	0    1    -1   0
-$EndComp
-$Comp
-L R R9
-U 1 1 585DBA25
-P 6400 2050
-F 0 "R9" V 6480 2050 50  0000 C CNN
-F 1 "120" V 6400 2050 50  0000 C CNN
-F 2 "Resistors_SMD:R_0805_HandSoldering" V 6330 2050 50  0001 C CNN
-F 3 "" H 6400 2050 50  0000 C CNN
-	1    6400 2050
 	0    1    -1   0
 $EndComp
@@
 DCD_4
 Wire Wire Line
-	6550 2050 6800 2050
-Wire Wire Line
-	6800 2150 6000 2150
-Wire Wire Line
 	6550 2250 6800 2250
 Wire Wire Line
@@
 Wire Wire Line
 	6550 2450 6800 2450
-Wire Wire Line
-	6800 2550 6000 2550
 Wire Wire Line
 	6550 2650 6800 2650
@@
 	0    -1   -1   0
 $EndComp
+Wire Wire Line
+	6000 2550 6800 2550
+NoConn ~ 6800 2050
+NoConn ~ 6800 2150
+NoConn ~ 9800 4050
+NoConn ~ 9800 4200
+Wire Wire Line
+	9500 4200 9800 4200
+Wire Wire Line
+	9800 4050 9500 4050
+Text Notes 9200 3950 0    60   ~ 0
+Ran out of GPIO outputs to control these pins
 $EndSCHEMATC
